File: Hardware/Spielmatte-PCB/Spielmatte-PCB.kicad_sch (KiCad schematic)
At the start: 60 parts, among them J1 USB_C_Receptacle, J2 Conn_01x04_Socket, Q1 2N3904, Q2 2N3904, SW1 SW_Push, SW10 SW_Push_45deg, SW11 SW_Push_45deg, SW12 SW_Push_45deg, SW13 SW_Push_45deg, SW14 SW_Push_45deg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

Commit message: Erweiterungen
Parts:
- added C10, C9: 22uF, symbol Device:C_Small
- added D18: LED, symbol Device:LED
- added R11: 10K, symbol Device:R_Small_US
- added R12: 1k, symbol Device:R_Small_US
- added U2: AMS1117-3.3, Package_TO_SOT_SMD:SOT-223-3_TabPin2, symbol Regulator_Linear:AMS1117-3.3
- R4: value 10k -> 0 OHm
Connections:
- net +3.3V: now also C10.1, D18.2 (A), R11.2, U2.2 (VO); no longer R4.2
- net +5V: now also C9.1, U2.3 (VI)
- net EN: now also U3.18 (~{RESET})
- net GND: now also U3.15 (A0), U3.16 (A1), U3.17 (A2), C10.2, C9.2, R12.1, U2.1 (GND); no longer D1.3 (DIN), R4.1, U1.7 (IO8)
- net SCL: now reaches U1.15 (IO3)
- net SCL: now also U3.12 (SCK)
- net SDA: now reaches U1.16 (IO2)
- net SDA: now also U3.13 (SDA)
- net INT B: now reaches U1.3 (IO4)
- net INT B: now also U3.19 (INTB)
- new net: D18.1 (K), R12.2
- new net: D1.3 (DIN), R4.1
- new net IO8: R11.1, R4.2, U1.7 (IO8)
- no-connect marks 34 -> 35
Other:
- note added: "DISPLAY CONNECTOR PINS"
- note added: "I2C PORTEXPANDER"
- note added: "POWER"
- note added: "RESET BOARD"
- note added: "RGB LED"
- note added: "TASTEN"
- note added: "USB CONNECTOR"
- note added: "USB to UART"
- moved on the sheet: C5, C6, C7, C8, D1, J2, R4, R5, R6, R7, R8, SW1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

Commit message: Update
Connections:
- net INT B: now also U1.4 (IO5); no longer U1.3 (IO4)
- net IO9: now also U1.8 (IO9); no longer U1.10 (IO10)
- net SCL: now also U1.3 (IO4); no longer U1.15 (IO3)
- net SCL_OLED: now also U1.6 (IO7); no longer U1.5 (IO6)
- net SDA: now also U1.15 (IO3); no longer U1.16 (IO2)
- net SDA_OLED: now also U1.5 (IO6); no longer U1.4 (IO5)
- no-connect marks 35 -> 41
Other:
- note added: "MAY NOT DELIVER ENOUGH POWER"
